File: Circuit design layout/Circuit design layout.sch (KiCad schematic (older format))
At the start: 0 parts

Commit message: changes
Parts:
- added R1: 1 MΩ, symbol Device:R
- added R2, R? (x9): 10 kΩ, symbol Device:R
- added RF? (x9): FSR, symbol misc_giogziro95:FSR
- added SW1: SW_Push_Open, symbol Switch:SW_Push_Open
- added U1: ATmega2560-16AU, Package_QFP:TQFP-100_14x14mm_P0.5mm, symbol MCU_Microchip_ATmega:ATmega2560-16AU
- added Y1: Resonator, symbol Device:Resonator
Connections:
- new net: SW1.2 (B), U1.30 (~RESET)
- new net: R1.2, U1.33 (XTAL2), Y1.3
- new net: R1.1, U1.34 (XTAL1), Y1.1
- new net: R2.1, SW1.1 (A)
- new net D2: U1.6 (PE4)
- new net D3: U1.7 (PE5)
- new net D4: U1.1 (PG5)
- new net Earth: R?.1, R?.1, R?.1, R?.1, R?.1, R?.1, R?.1, R?.1, R?.1, U1.11 (GND), U1.32 (GND), U1.62 (GND), U1.81 (GND), U1.99 (GND), Y1.2
- new net FSR0: R?.2, RF?.1, U1.97 (PF0)
- new net FSR1: R?.2, RF?.1, U1.96 (PF1)
- new net FSR2: R?.2, RF?.1, U1.95 (PF2)
- new net FSR3: R?.2, RF?.1, U1.94 (PF3)
- new net FSR4: R?.2, RF?.1, U1.93 (PF4)
- new net FSR5: R?.2, RF?.1, U1.92 (PF5)
- new net FSR6: R?.2, RF?.1, U1.91 (PF6)
- new net FSR7: R?.2, RF?.1, U1.90 (PF7)
- new net FSR8: R?.2, RF?.1, U1.89 (PK0)
- new net VCC: R2.2, RF?.2, RF?.2, RF?.2, RF?.2, RF?.2, RF?.2, RF?.2, RF?.2, RF?.2, U1.10 (VCC), U1.100 (AVCC), U1.31 (VCC), U1.61 (VCC), U1.80 (VCC)
- no-connect marks 0 -> 7
